File: Calculator/Calculator.kicad_sch (KiCad schematic)
At the start: 0 parts

Commit message: :memo: Added esp32wroom
Parts:
- added C1, C2: 100nF, Capacitor_Tantalum_SMD:CP_EIA-3216-18_Kemet-A, symbol Device:C
- added C8: 100nF, symbol Device:C
- added C9: 10nF, symbol Device:C
- added D1: SS36, Diode_THT:D_DO-35_SOD27_P7.62mm_Horizontal, symbol Diode:1N6857
- added D2: LED, LED_SMD:LED_Cree-XP, symbol Device:LED
- added E2: 100uF/35V, Capacitor_SMD:C_1808_4520Metric_Pad1.72x2.30mm_HandSolder, symbol Device:C_Polarized_Small_US
- added E3, E4: 220uF/10V, Capacitor_SMD:C_1808_4520Metric_Pad1.72x2.30mm_HandSolder, symbol Device:C_Polarized_Small_US
- added L1: 68uF/2A, Inductor_SMD:L_Sunlord_MWSA0605S, symbol Device:L
- added R1: 1K, Resistor_SMD:R_1206_3216Metric, symbol Device:R
- added R2: 10K, symbol Device:R
- added R3, R4: R, symbol Device:R
- added SW1, SW2: SW_Push, symbol Switch:SW_Push
- added U1: XL1509-5.0, Package_SO:SOIC-8_3.9x4.9mm_P1.27mm, symbol Regulator_Switching:XL1509-5.0
- added U2: AMS1117-3.3, Package_TO_SOT_SMD:SOT-223-3_TabPin2, symbol Regulator_Linear:AMS1117-3.3
- added U3: ESP32-WROOM-32E(4MB), ESP32-WROOM-32E-N4:WIFI-SMD_ESP32-WROOM-32E, symbol ESP32-WROOM-32E-N4:ESP32-WROOM-32E(4MB)
Connections:
- new net: R3.2, U3.25 (IO0)
- new net: R2.1, SW1.2
- new net: D2.2 (A), R1.2
- new net +12V: E2.1
- new net +3.3V: C8.2, C9.2, R2.2, R3.1, R4.2, SW2.1, U3.2 (3V3), U3.23 (IO15), U3.3 (EN)
- new net -12V: U1.1 (VIN)
- new net -3.3V: C2.2, E4.1, R1.1, U2.2 (VO)
- new net 1025: U3.10 (IO25)
- new net 1026: U3.11 (IO26)
- new net 1027: U3.12 (IO27)
- new net CS: U3.29 (IO5)
- new net GND: C1.2, C2.1, C8.1, C9.1, D1.2 (A), D2.1 (K), E2.2, E3.2, E4.2, R4.1, SW1.1, SW2.2, U1.4 (~{EN}), U1.5 (GND), U1.6 (GND), U1.7 (GND), U1.8 (GND), U2.1 (GND), U3.1 (GND), U3.38 (GND), U3.39 (GND)
- new net IO12: U3.14 (IO12)
- new net IO13: U3.16 (IO13)
- new net IO14: U3.13 (IO14)
- new net IO16: U3.27 (IO16)
- new net IO17: U3.28 (IO17)
- new net IO2: U3.24 (IO2)
- new net IO32: U3.8 (IO32)
- new net IO33: U3.9 (IO33)
- new net IO34: U3.6 (IO34)
- new net IO35: U3.7 (IO35)
- new net IO4: U3.26 (IO4)
- new net MISO: U3.31 (IO19)
- new net MOSI: U3.37 (IO23)
- new net OUT 5V: D1.1 (K), L1.1, U1.2 (OUT)
- new net RXD0: U3.34 (RXD0)
- new net SCK: U3.30 (IO18)
- new net SCL: U3.36 (IO22)
- new net SDA: U3.33 (IO21)
- new net SENSOR_VN: U3.5 (SENSOR_VN)
- new net SENSOR_VP: U3.4 (SENSOR_VP)
- new net TXD0: U3.35 (TXD0)
- new net VCC: C1.1, E3.1, L1.2, U1.3 (FB), U2.3 (VI)
- no-connect marks 0 -> 8
Other:
- note added: "ESP32_WROOM"
- note added: "LDO/ POWER"
